File: Arduino_clone.kicad_sch (KiCad schematic)
At the start: 13 parts, among them U1 DS1337_ben, U2 24LC1025, U3 24LC1025, U4 ATmega328P-A, Y1 Crystal, Y2 Crystal

Commit message: connceting wires together before DRC
Parts:
- R1: value R -> 330ohm
Connections:
- net GND is gone; now on net GNDPWR: U4.21 (GND), U4.3 (GND), U4.5 (GND)
- net D2: now also U4.32 (PD2)
- net D3: now also U4.1 (PD3)
- net D4: now also U4.2 (PD4)
- net D5: now also U4.9 (PD5)
- net D6: now also U4.10 (PD6)
- net D7: now also U4.11 (PD7)
- net D8: now also U4.12 (PB0)
- net RX: now also U4.30 (PD0)
- net SDA: now also U1.5 (SDA), U2.5 (SDA), U3.5 (SDA), U4.27 (PC4)
- net TX: now also U4.31 (PD1)
- net reset: now also R2.2
- net sck: now also D1.2 (A), U1.6 (SCL), U2.6 (SCL), U3.6 (SCL)
- net vcc: now also BT1.1 (+), C3.1, R2.1, U1.3 (INTA), U1.8 (vcc), U2.3 (A2), U2.8 (VCC), U3.3 (A2), U3.8 (VCC), U4.20 (AREF)
- net GNDPWR: now reaches C2.1
- net GNDPWR: now also BT1.2 (-), C1.1, C3.2, R1.2, U1.4 (GND), U2.4 (GND), U2.7 (WP), U3.4 (GND), U3.7 (WP)
- net at C2.2: now also U4.7 (XTAL1/PB6), Y2.2
- net at Y2.1: now also C1.2, U4.8 (XTAL2/PB7)
- net ADDS1: now reaches U3.1 (A0)
- net ADDS1: now also U2.1 (A0), U4.23 (PC0)
- net ADDS2: now reaches U3.2 (A1)
- net ADDS2: now also U2.2 (A1), U4.24 (PC1)
- net at Y1.1: now also U1.1 (X1)
- net at Y1.2: now also U1.2 (X2)
- net at D1.1 (K): now also R1.1
- no-connect marks 0 -> 8
Other:
- sheet connectors ports: added none; removed SCKIC2
- moved on the sheet: BT1, C1, C2, C3, D1, R1, R2, U2, U3, Y1, Y2

Commit message: set design rules and loaded component for pcb new
Connections:
- net vcc: no longer BT1.1 (+), C3.1, R2.1, U1.3 (INTA), U1.8 (vcc), U2.3 (A2), U2.8 (VCC), U3.3 (A2), U3.8 (VCC), U4.18 (AVCC), U4.4 (VCC), U4.6 (VCC)
- new net VCC: BT1.1 (+), C3.1, R2.1, U1.3 (INTA), U1.8 (vcc), U2.3 (A2), U2.8 (VCC), U3.3 (A2), U3.8 (VCC), U4.18 (AVCC), U4.4 (VCC), U4.6 (VCC)
Changed lines of the file:
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@@
   (junction (at 58.42 132.08) (diameter 0) (color 0 0 0 0)
   )
+  (junction (at 214.63 111.76) (diameter 0) (color 0 0 0 0)
+  )
   (junction (at 184.15 109.22) (diameter 0) (color 0 0 0 0)
   )
@@
   (junction (at 63.5 132.08) (diameter 0) (color 0 0 0 0)
   )
+  (junction (at 68.58 110.49) (diameter 0) (color 0 0 0 0)
+  )
   (junction (at 184.15 111.76) (diameter 0) (color 0 0 0 0)
   )
@@
   (junction (at 242.57 80.01) (diameter 0) (color 0 0 0 0)
   )
-  (no_connect (at 170.18 66.04))
   (no_connect (at 170.18 71.12))
   (no_connect (at 170.18 73.66))
+  (no_connect (at 170.18 66.04))
   (no_connect (at 170.18 96.52))
   (no_connect (at 170.18 99.06))
@@
     (stroke (width 0) (type default) (color 0 0 0 0))
   )
-  (wire (pts (xy 48.26 110.49) (xy 78.74 110.49))
+  (wire (pts (xy 48.26 110.49) (xy 68.58 110.49))
     (stroke (width 0) (type default) (color 0 0 0 0))
   )
@@
     (stroke (width 0) (type default) (color 0 0 0 0))
   )
+  (wire (pts (xy 214.63 111.76) (xy 224.79 111.76))
+    (stroke (width 0) (type default) (color 0 0 0 0))
+  )
   (wire (pts (xy 91.44 58.42) (xy 102.87 58.42))
     (stroke (width 0) (type default) (color 0 0 0 0))
@@
     (stroke (width 0) (type default) (color 0 0 0 0))
   )
-  (wire (pts (xy 184.15 111.76) (xy 224.79 111.76))
+  (wire (pts (xy 184.15 111.76) (xy 214.63 111.76))
     (stroke (width 0) (type default) (color 0 0 0 0))
   )
@@
     (stroke (width 0) (type default) (color 0 0 0 0))
   )
+  (wire (pts (xy 68.58 110.49) (xy 78.74 110.49))
+    (stroke (width 0) (type default) (color 0 0 0 0))
+  )
   (wire (pts (xy 161.29 63.5) (xy 170.18 63.5))
     (stroke (width 0) (type default) (color 0 0 0 0))
@@
     (effects (font (size 1.27 1.27)) (justify left bottom))
   )
-  (label "vcc" (at 38.1 124.46 180)
+  (label "VCC" (at 38.1 124.46 180)
     (effects (font (size 1.27 1.27)) (justify right bottom))
   )
@@
     (effects (font (size 1.27 1.27)) (justify right bottom))
   )
-  (label "vcc" (at 64.77 110.49 180)
+  (label "VCC" (at 64.77 110.49 180)
     (effects (font (size 1.27 1.27)) (justify right bottom))
   )
@@
     (effects (font (size 1 1)) (justify right bottom))
   )
-  (label "vcc" (at 161.29 55.88 90)
+  (label "VCC" (at 161.29 55.88 90)
     (effects (font (size 1.27 1.27)) (justify left bottom))
   )
@@
     (effects (font (size 1.27 1.27)) (justify right bottom))
   )
-  (label "vcc" (at 101.6 172.72 180)
+  (label "VCC" (at 101.6 172.72 180)
     (effects (font (size 1.27 1.27)) (justify right bottom))
   )
@@
     (effects (font (size 1.27 1.27)) (justify left bottom))
   )
-  (label "vcc" (at 68.58 124.46 180)
+  (label "VCC" (at 68.58 124.46 180)
     (effects (font (size 1.27 1.27)) (justify right bottom))
   )
@@
     (effects (font (size 1.27 1.27)) (justify right bottom))
   )
-  (label "vcc" (at 184.15 116.84 270)
-    (effects (font (size 1.27 1.27)) (justify right bottom))
-  )
-  (label "vcc" (at 43.18 69.85 180)
-    (effects (font (size 1.27 1.27)) (justify right bottom))
-  )
-  (label "D8" (at 151.13 184.15 0)
+  (label "VCC" (at 184.15 116.84 270)
+    (effects (font (size 1.27 1.27)) (justify right bottom))
+  )
+  (label "VCC" (at 43.18 69.85 180)
+    (effects (font (size 1.27 1.27)) (justify right bottom))
+  )
+  (label "D8" (at 149.86 184.15 0)
     (effects (font (size 1.27 1.27)) (justify left bottom))
   )
@@
     (effects (font (size 1.27 1.27)) (justify right bottom))
   )
-  (label "vcc" (at 53.34 57.15 90)
+  (label "VCC" (at 53.34 57.15 90)
     (effects (font (size 1.27 1.27)) (justify left bottom))
   )
@@
     (pin "2")
   )
+  (symbol (lib_id "power:PWR_FLAG") (at 214.63 111.76 0) (unit 1)
+    (in_bom yes) (on_board yes) (fields_autoplaced)
+    (property "Reference" "#FLG0101" (id 0) (at 214.63 109.855 0)
+      (effects (font (size 1.27 1.27)) hide)
+    )
+    (property "Value" "PWR_FLAG" (id 1) (at 214.63 106.68 0))
+    (property "Footprint" "" (id 2) (at 214.63 111.76 0)
+      (effects (font (size 1.27 1.27)) hide)
+    )
+    (property "Datasheet" "~" (id 3) (at 214.63 111.76 0)
+      (effects (font (size 1.27 1.27)) hide)
+    )
+    (pin "1")
+  )
   (symbol (lib_id "Device:Crystal") (at 134.62 57.15 270) (unit 1)
     (in_bom yes) (on_board yes) (fields_autoplaced)
@@
   (symbol (lib_id "power:GNDPWR") (at 63.5 132.08 0) (unit 1)
     (in_bom yes) (on_board yes) (fields_autoplaced)
-    (property "Reference" "#PWR?" (id 0) (at 63.5 137.16 0)
+    (property "Reference" "#PWR0103" (id 0) (at 63.5 137.16 0)
       (effects (font (size 1.27 1.27)) hide)
     )
@@
   (symbol (lib_id "power:GNDPWR") (at 242.57 81.28 0) (unit 1)
     (in_bom yes) (on_board yes) (fields_autoplaced)
-    (property "Reference" "#PWR?" (id 0) (at 242.57 86.36 0)
+    (property "Reference" "#PWR0107" (id 0) (at 242.57 86.36 0)
       (effects (font (size 1.27 1.27)) hide)
     )
@@
     (pin "1")
     (pin "2")
+  )
+  (symbol (lib_id "power:PWR_FLAG") (at 68.58 110.49 0) (unit 1)
+    (in_bom yes) (on_board yes) (fields_autoplaced)
+    (property "Reference" "#FLG?" (id 0) (at 68.58 108.585 0)
+      (effects (font (size 1.27 1.27)) hide)
+    )
+    (property "Value" "PWR_FLAG" (id 1) (at 68.58 105.41 0))
+    (property "Footprint" "" (id 2) (at 68.58 110.49 0)
+      (effects (font (size 1.27 1.27)) hide)
+    )
+    (property "Datasheet" "~" (id 3) (at 68.58 110.49 0)
+      (effects (font (size 1.27 1.27)) hide)
+    )
+    (pin "1")
   )
   (symbol (lib_id "Device:R") (at 161.29 59.69 0) (unit 1)
@@
   (symbol (lib_id "power:GNDPWR") (at 53.34 74.93 0) (unit 1)
     (in_bom yes) (on_board yes) (fields_autoplaced)
-    (property "Reference" "#PWR?" (id 0) (at 53.34 80.01 0)
+    (property "Reference" "#PWR0102" (id 0) (at 53.34 80.01 0)
       (effects (font (size 1.27 1.27)) hide)
     )
@@
   (symbol (lib_id "power:GNDPWR") (at 120.65 102.87 0) (unit 1)
     (in_bom yes) (on_board yes) (fields_autoplaced)
-    (property "Reference" "#PWR?" (id 0) (at 120.65 107.95 0)
+    (property "Reference" "#PWR0104" (id 0) (at 120.65 107.95 0)
       (effects (font (size 1.27 1.27)) hide)
     )
@@
   (symbol (lib_id "power:GNDPWR") (at 175.26 29.21 0) (unit 1)
     (in_bom yes) (on_board yes) (fields_autoplaced)
-    (property "Reference" "#PWR?" (id 0) (at 175.26 34.29 0)
+    (property "Reference" "#PWR0106" (id 0) (at 175.26 34.29 0)
       (effects (font (size 1.27 1.27)) hide)
     )
@@
   (symbol (lib_id "power:GNDPWR") (at 91.44 58.42 0) (unit 1)
     (in_bom yes) (on_board yes) (fields_autoplaced)
-    (property "Reference" "#PWR?" (id 0) (at 91.44 63.5 0)
+    (property "Reference" "#PWR0105" (id 0) (at 91.44 63.5 0)
       (effects (font (size 1.27 1.27)) hide)
     )
@@
   )
   (symbol_instances
+    (path "/2a6309ac-1c78-47ff-b8d2-6ffea4db9b2f"
+      (reference "#FLG0101") (unit 1) (value "PWR_FLAG") (footprint "")
+    )
+    (path "/b63d5690-5d29-4544-98ef-112a3c40f96b"
+      (reference "#FLG?") (unit 1) (value "PWR_FLAG") (footprint "")
+    )
     (path "/5202d06b-b768-4eb0-821f-d3af277798e2"
       (reference "#PWR0101") (unit 1) (value "GNDPWR") (footprint "")
     )
+    (path "/d94c5a20-85f6-4d1a-a831-12e6e9755b99"
+      (reference "#PWR0102") (unit 1) (value "GNDPWR") (footprint "")
+    )
     (path "/4b0111fa-a5f2-44e5-80bd-d8311a11ed82"
-      (reference "#PWR?") (unit 1) (value "GNDPWR") (footprint "")
+      (reference "#PWR0103") (unit 1) (value "GNDPWR") (footprint "")
+    )
+    (path "/de89a706-ecec-4d5e-b372-50bf4c84c7dc"
+      (reference "#PWR0104") (unit 1) (value "GNDPWR") (footprint "")
+    )
+    (path "/ec3b3571-8083-4056-ba3b-107778b0c07b"
+      (reference "#PWR0105") (unit 1) (value "GNDPWR") (footprint "")
+    )
+    (path "/e5c557f7-4781-4a7b-bb01-1b654de21101"
+      (reference "#PWR0106") (unit 1) (value "GNDPWR") (footprint "")
     )
     (path "/906159d3-a2fe-4c74-8f6f-7fb7036a106b"
-      (reference "#PWR?") (unit 1) (value "GNDPWR") (footprint "")
-    )
-    (path "/d94c5a20-85f6-4d1a-a831-12e6e9755b99"
-      (reference "#PWR?") (unit 1) (value "GNDPWR") (footprint "")
-    )
-    (path "/de89a706-ecec-4d5e-b372-50bf4c84c7dc"
-      (reference "#PWR?") (unit 1) (value "GNDPWR") (footprint "")
-    )
-    (path "/e5c557f7-4781-4a7b-bb01-1b654de21101"
-      (reference "#PWR?") (unit 1) (value "GNDPWR") (footprint "")
-    )
-    (path "/ec3b3571-8083-4056-ba3b-107778b0c07b"
-      (reference "#PWR?") (unit 1) (value "GNDPWR") (footprint "")
+      (reference "#PWR0107") (unit 1) (value "GNDPWR") (footprint "")
     )
     (path "/19cd3de1-faa9-409c-93a7-570d16f1bc1e"
