File: Arduino_clone4_layer.kicad_pcb (KiCad board)
At the start: 4 copper layers, 41 x 30 mm, 17 parts, among them J1 Conn_01x04, J2 DIGITAL PIN, J3 Conn_01x04, J4 icsp, U1 DS1337_ben, U2 24LC1025, U3 24LC1025, U4 ATmega328P-A, Y1 Crystal, Y2 Crystal

Commit message: copper fillxone on the 2layer boared
Routing:
- added copper zone on In2.Cu, net GNDPWR
Changed lines of the file:
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@@
   (segment (start 134.1728 93.9042) (end 134.1728 95.0795) (width 0.25) (layer "B.Cu") (net 32))
   (segment (start 138.89 99.7967) (end 138.89 117.62) (width 0.25) (layer "B.Cu") (net 32))
+  (zone (net 2) (net_name "GNDPWR") (layer "In2.Cu") (hatch edge 0.508)
+    (connect_pads (clearance 0.508))
+    (min_thickness 0.254) (filled_areas_thickness no)
+    (fill yes (thermal_gap 0.508) (thermal_bridge_width 0.508))
+    (polygon
+      (pts
+        (xy 146.0754 91.4654)
+        (xy 146.4818 91.5416)
+        (xy 146.3548 91.5416)
+        (xy 146.3548 120.4214)
+        (xy 106.5784 120.4214)
+        (xy 106.68 91.4146)
+      )
+    )
+  )
 )
